File: control/control.kicad_pcb (KiCad board)
At the start: 2 copper layers, 100 x 50 mm, 64 parts, among them J101 Conn_02x03_Odd_Even, J103 USART, J104 ENCODER, J105 SWITCHES, J106 POSITION, J107 DEBUG, J401 RJ45_Shielded, J402 RJ45_Shielded, SW102 CENTER_SW, U201 STM32L431RCTx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

Commit message: Add UV fab files
Parts:
- removed H101, H102, H103, H104: MountingHole, MountingHole:MountingHole_3.2mm_M3
- added ?: , , F.Cu at (176.8, 103.7)
- added ?: , , F.Cu at (85.3, 103.7)
- added ?: , , F.Cu at (85.2, 62.3)
- added ?: , , F.Cu at (176.8, 62.3)
Routing:
- net +15V: track 49.4 -> 62.7 mm
- net GND: track 528.3 -> 537.0 mm
- net unconnected-(U201-PH0-Pad5): track 5.37 -> 0.00 mm
- net /can_connector/CAN_18V: track 45.7 -> 49.1 mm
- net /ADC_INPUT_VOLTAGE: track 66.2 -> 65.0 mm
