File: control/stm32.kicad_sch (KiCad schematic)
At the start: 18 parts, among them U201 STM32L431RCTx

Commit message: Add UV fab files
Connections:
- no-connect marks 27 -> 28
Other:
- note added: "6 x 100nF"
- note removed: "5 x 100nF"
Changed lines of the file:
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@@
 (kicad_sch
-	(version 20231120)
+	(version 20250114)
 	(generator "eeschema")
-	(generator_version "8.0")
+	(generator_version "9.0")
 	(paper "A4")
+	(text "6 x 100nF"
+		(exclude_from_sim no)
+		(at 73.66 72.39 0)
+		(effects
+			(font
+				(size 1.016 1.016)
+			)
+			(justify left bottom)
+		)
+	)
 	(junction
 		(at 62.23 53.34)
@@
 	)
 	(junction
+		(at 120.65 74.93)
+		(diameter 0)
+		(color 0 0 0 0)
+	)
+	(junction
 		(at 100.33 60.96)
 		(diameter 0)
@@
 	)
 	(junction
-		(at 118.11 74.93)
-		(diameter 0)
-		(color 0 0 0 0)
-	)
-	(junction
 		(at 107.95 74.93)
 		(diameter 0)
@@
 	)
 	(no_connect
+		(at 85.09 111.76)
+	)
+	(no_connect
 		(at 118.11 157.48)
 	)
@@
 	(wire
 		(pts
-			(xy 118.11 71.12) (xy 118.11 74.93)
+			(xy 120.65 71.12) (xy 120.65 74.93)
 		)
 		(stroke
@@
 	(polyline
 		(pts
-			(xy 60.96 72.39) (xy 82.55 72.39)
+			(xy 55.88 72.39) (xy 82.55 72.39)
 		)
 		(stroke
@@
 	(wire
 		(pts
-			(xy 115.57 74.93) (xy 118.11 74.93)
+			(xy 115.57 74.93) (xy 120.65 74.93)
 		)
 		(stroke
@@
 	(polyline
 		(pts
-			(xy 82.55 64.77) (xy 60.96 64.77)
+			(xy 82.55 64.77) (xy 55.88 64.77)
 		)
 		(stroke
@@
 	(wire
 		(pts
-			(xy 115.57 71.12) (xy 118.11 71.12)
+			(xy 115.57 71.12) (xy 120.65 71.12)
 		)
 		(stroke
@@
 	(polyline
 		(pts
-			(xy 60.96 72.39) (xy 60.96 72.39)
+			(xy 55.88 72.39) (xy 60.96 72.39)
 		)
 		(stroke
@@
 	(polyline
 		(pts
-			(xy 60.96 64.77) (xy 60.96 72.39)
+			(xy 55.88 64.77) (xy 55.88 72.39)
 		)
 		(stroke
@@
 		)
 	)
-	(wire
-		(pts
-			(xy 118.11 74.93) (xy 120.65 74.93)
-		)
-		(stroke
-			(width 0)
-			(type default)
-		)
-	)
-	(text "5 x 100nF"
-		(exclude_from_sim no)
-		(at 73.66 72.39 0)
-		(effects
-			(font
-				(size 1.016 1.016)
-			)
-			(justify left bottom)
-		)
-	)
 	(label "RED_LED"
 		(at 209.55 113.03 0)
@@
 		(dnp no)
 		(property "Reference" "C205"
-			(at 70.485 66.04 0)
+			(at 82.804 71.12 0)
 			(effects
 				(font
@@
 		(dnp no)
 		(property "Reference" "C207"
-			(at 78.105 66.04 0)
+			(at 82.804 75.438 0)
 			(effects
 				(font
@@
 		(dnp no)
 		(property "Reference" "C208"
-			(at 123.19 73.025 90)
+			(at 124.46 72.898 90)
 			(effects
 				(font
@@
 		(dnp no)
 		(property "Reference" "C201"
-			(at 55.245 75.565 90)
+			(at 53.086 77.978 90)
 			(effects
 				(font
@@
 		)
 		(property "Value" "25V 10uF X5R ±10% 0805"
-			(at 55.245 72.39 90)
+			(at 53.086 72.644 90)
 			(effects
 				(font
@@
 		(dnp no)
 		(property "Reference" "R202"
-			(at 54.5084 119.38 90)
+			(at 46.736 120.65 90)
 			(effects
 				(font
@@
 		)
 		(property "Value" "10kR 0805"
-			(at 52.197 119.38 90)
+			(at 43.942 121.412 90)
 			(effects
 				(font
@@
 		(dnp no)
 		(property "Reference" "C206"
-			(at 74.93 66.04 0)
+			(at 82.804 73.152 0)
 			(effects
 				(font
@@
 		(dnp no)
 		(property "Reference" "R201"
-			(at 54.61 113.03 90)
+			(at 44.196 111.506 90)
 			(effects
 				(font
@@
 		)
 		(property "Value" "BOOT0"
-			(at 52.07 113.03 90)
+			(at 46.482 111.506 90)
 			(effects
 				(font
