File: hardware/power/Switches.kicad_pcb (KiCad board)
At the start: 2 copper layers, 100 x 50 mm, 71 parts, among them J101 Screw_Terminal_01x02, J102 Screw_Terminal_01x02, J105 Conn_02x03_Odd_Even, Q101 BSC093N15NS5, Q104 BSC093N15NS5, Q107 BSC093N15NS5, Q110 BSC093N15NS5, U101 UCC27211DDAR, U102 UCC27211DDAR, U105 INA283

Commit message: Organize schematics per domain
Parts:
- removed H112, H114, H116: MountingHole, MountingHole:MountingHole_3.5mm_Pad
